File: KF1950.kicad_sch (KiCad schematic)
At the start: 51 parts, among them Q1 MMBT3906, U5 SPX3819M5-L-1-8, U7 25MHz, U9 SN74AVC4T774

Commit message: All components placed
Went through TI schematic and layout checklist.
All components placed and initial DRC
Need thermal vias on KF1950 and also better layout (so not so many errors)
Need to do silk
Parts:
- removed R18, R20: 0, Resistor_SMD:R_0402_1005Metric, symbol Device:R_US
- removed TP29, TP30, TP31, TP32, TP33, TP34: TestPoint, TestPoint:TestPoint_Pad_D1.5mm, symbol Connector:TestPoint
- added R79: 0, Resistor_SMD:R_0402_1005Metric, symbol Device:R_US
- added RST_DET1, TP12, TP13, TP14, TP15, TP16, TP17, TP18: TestPoint, TestPoint:TestPoint_Pad_D1.5mm, symbol Connector:TestPoint
- added TP20, TP21, TP23, TP24, TP25, TP26: TestPoint, TestPoint:TestPoint_Pad_D1.0mm, symbol Connector:TestPoint
- R32: value 390 -> 400
- R33: value 27.5 -> 33
- R34: value 33 -> 27
- U7: value 25MHz -> 24MHz
Connections:
- net 1V2 is gone; now on net 1V8: C29.2, U7.4 (VIN)
- net 1V8: no longer C28.1, R32.2
- net ESP_RXD: no longer R17.1
- net GND: now also C28.1, R17.1, R32.2, TP17.1; no longer C26.2, C30.2, U5.2 (GND), U9.6 (A4)
- net LDO_GND: now also C26.2, C30.2, U5.2 (GND)
- net RST_DET: now also RST_DET1.1
- net RST_N_1V8: now also TP15.1
- net RXD: now also TP13.1
- net RXD_1V8: now also R79.1
- net TXD: now also R79.2, TP12.1; no longer R17.2
- net TXD_1V8: now also TP16.1
- net /RST: now also TP14.1
- net at U8.12 (GND): now also TP26.1
- net at U8.13 (DIR): now also TP25.1
- net at U8.15 (0.9V): now also TP24.1
- net at U8.17 (RXD): now also TP23.1
- net at U8.18 (CTSI): now also TP21.1
- net at U8.20 (CLK): now also TP20.1
- net at U9.11 (B4): now also TP18.1
- new net: R17.2, U9.6 (A4)
- no-connect marks 9 -> 1
Other:
- note added: "Watch how TXD/RXD move from perspective of ESP to ASIC As per Hashboards, level shifter is only needed for ASIC TXD ( 1.8V -> 3.3V)"
- note removed: "Check this CTI to GND"
- note removed: "Check this RC circuit"
- moved on the sheet: C26, C28, C30, C33, C34, C47, R19, R26, R27, R28, R29, R30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

Commit message: Silk Done
Still need to fix up heatsink vias on ASIC and paste layer for thermal
Parts:
- renumbered TP24 to 0.9V, TP19 to 1V8, TP21 to CTSI, TP25 to DIR_HI, TP26 to DIR_LO, TP14 to RST, TP15 to RST_LO, TP13 to RXD, TP23 to RXD, TP18 to TP_HI, TP17 to TP_LO, TP20 to TXD, TP12 to TXD, TP16 to TXD_LO
Other:
- moved on the sheet: TXD
Changed lines of the file:
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@@
 	(wire
 		(pts
+			(xy 173.99 104.14) (xy 172.72 104.14)
+		)
+		(stroke
+			(width 0)
+			(type default)
+		)
+	)
+	(wire
+		(pts
 			(xy 38.1 31.75) (xy 39.37 31.75)
 		)
@@
 	(symbol
 		(lib_id "Connector:TestPoint")
-		(at 172.72 104.14 270)
+		(at 173.99 104.14 270)
 		(unit 1)
 		(exclude_from_sim no)
@@
 		(on_board yes)
 		(dnp no)
-		(fields_autoplaced yes)
-		(property "Reference" "TP20"
-			(at 177.8 102.8699 90)
+		(property "Reference" "TXD"
+			(at 177.8 104.14 90)
 			(effects
 				(font
@@
 		)
 		(property "Value" "TestPoint"
-			(at 177.8 105.4099 90)
+			(at 179.07 105.4099 90)
 			(effects
 				(font
@@
 				)
 				(justify left)
+				(hide yes)
 			)
 		)
 		(property "Footprint" "TestPoint:TestPoint_Pad_D1.0mm"
-			(at 172.72 109.22 0)
+			(at 173.99 109.22 0)
 			(effects
 				(font
@@
 		)
 		(property "Datasheet" "~"
-			(at 172.72 109.22 0)
+			(at 173.99 109.22 0)
 			(effects
 				(font
@@
 		)
 		(property "Description" "test point"
-			(at 172.72 104.14 0)
+			(at 173.99 104.14 0)
 			(effects
 				(font
@@
 			(project ""
 				(path "/e63e39d7-6ac0-4ffd-8aa3-1841a4541b55/4cf9c075-d009-4c35-9949-adda70ae20c7"
-					(reference "TP20")
+					(reference "TXD")
 					(unit 1)
 				)
@@
 		(on_board yes)
 		(dnp no)
-		(property "Reference" "TP14"
+		(property "Reference" "RST"
 			(at 62.23 116.84 90)
 			(effects
@@
 			(project "BitshokaNiniV1.1"
 				(path "/e63e39d7-6ac0-4ffd-8aa3-1841a4541b55/4cf9c075-d009-4c35-9949-adda70ae20c7"
-					(reference "TP14")
+					(reference "RST")
 					(unit 1)
 				)
@@
 		(on_board yes)
 		(dnp no)
-		(property "Reference" "TP13"
+		(property "Reference" "RXD"
 			(at 62.23 109.22 90)
 			(effects
@@
 			(project "BitshokaNiniV1.1"
 				(path "/e63e39d7-6ac0-4ffd-8aa3-1841a4541b55/4cf9c075-d009-4c35-9949-adda70ae20c7"
-					(reference "TP13")
+					(reference "RXD")
 					(unit 1)
 				)
@@
 		(on_board yes)
 		(dnp no)
-		(fields_autoplaced yes)
-		(property "Reference" "TP24"
-			(at 177.8 115.5699 90)
+		(property "Reference" "0.9V"
+			(at 177.8 116.84 90)
 			(effects
 				(font
@@
 				)
 				(justify left)
+				(hide yes)
 			)
 		)
@@
 			(project "BitshokaNiniV1.1"
 				(path "/e63e39d7-6ac0-4ffd-8aa3-1841a4541b55/4cf9c075-d009-4c35-9949-adda70ae20c7"
-					(reference "TP24")
+					(reference "0.9V")
 					(unit 1)
 				)
@@
 		(on_board yes)
 		(dnp no)
-		(fields_autoplaced yes)
-		(property "Reference" "TP21"
-			(at 177.8 107.9499 90)
+		(property "Reference" "CTSI"
+			(at 177.8 109.22 90)
 			(effects
 				(font
@@
 				)
 				(justify left)
+				(hide yes)
 			)
 		)
@@
 			(project "BitshokaNiniV1.1"
 				(path "/e63e39d7-6ac0-4ffd-8aa3-1841a4541b55/4cf9c075-d009-4c35-9949-adda70ae20c7"
-					(reference "TP21")
+					(reference "CTSI")
 					(unit 1)
 				)
@@
 		(on_board yes)
 		(dnp no)
-		(fields_autoplaced yes)
-		(property "Reference" "TP26"
-			(at 177.8 123.1899 90)
+		(property "Reference" "DIR_LO"
+			(at 177.8 124.46 90)
 			(effects
 				(font
@@
 				)
 				(justify left)
+				(hide yes)
 			)
 		)
@@
 			(project "BitshokaNiniV1.1"
 				(path "/e63e39d7-6ac0-4ffd-8aa3-1841a4541b55/4cf9c075-d009-4c35-9949-adda70ae20c7"
-					(reference "TP26")
+					(reference "DIR_LO")
 					(unit 1)
 				)
@@
 		(on_board yes)
 		(dnp no)
-		(fields_autoplaced yes)
-		(property "Reference" "TP25"
-			(at 177.8 120.6499 90)
+		(property "Reference" "DIR_HI"
+			(at 177.8 121.92 90)
 			(effects
 				(font
@@
 				)
 				(justify left)
+				(hide yes)
 			)
 		)
@@
 			(project "BitshokaNiniV1.1"
 				(path "/e63e39d7-6ac0-4ffd-8aa3-1841a4541b55/4cf9c075-d009-4c35-9949-adda70ae20c7"
-					(reference "TP25")
+					(reference "DIR_HI")
 					(unit 1)
 				)
@@
 		(on_board yes)
 		(dnp no)
-		(fields_autoplaced yes)
-		(property "Reference" "TP23"
-			(at 177.8 110.4899 90)
+		(property "Reference" "RXD"
+			(at 177.8 111.76 90)
 			(effects
 				(font
@@
 				)
 				(justify left)
+				(hide yes)
 			)
 		)
@@
 			(project "BitshokaNiniV1.1"
 				(path "/e63e39d7-6ac0-4ffd-8aa3-1841a4541b55/4cf9c075-d009-4c35-9949-adda70ae20c7"
-					(reference "TP23")
+					(reference "RXD")
 					(unit 1)
 				)
@@
 		(on_board yes)
 		(dnp no)
-		(property "Reference" "TP15"
-			(at 187.96 33.02 90)
+		(property "Reference" "RST_LO"
+			(at 186.69 33.02 90)
 			(effects
 				(font
@@
 			(project "BitshokaNiniV1.1"
 				(path "/e63e39d7-6ac0-4ffd-8aa3-1841a4541b55/4cf9c075-d009-4c35-9949-adda70ae20c7"
-					(reference "TP15")
+					(reference "RST_LO")
 					(unit 1)
 				)
@@
 		(on_board yes)
 		(dnp no)
-		(property "Reference" "TP19"
+		(property "Reference" "1V8"
 			(at 67.31 29.21 90)
 			(effects
@@
 			(project "BitshokaNiniV1.1"
 				(path "/e63e39d7-6ac0-4ffd-8aa3-1841a4541b55/4cf9c075-d009-4c35-9949-adda70ae20c7"
-					(reference "TP19")
+					(reference "1V8")
 					(unit 1)
 				)
@@
 		(on_board yes)
 		(dnp no)
-		(property "Reference" "TP17"
-			(at 187.96 40.64 90)
+		(property "Reference" "TP_LO"
+			(at 186.69 40.64 90)
 			(effects
 				(font
@@
 			(project "BitshokaNiniV1.1"
 				(path "/e63e39d7-6ac0-4ffd-8aa3-1841a4541b55/4cf9c075-d009-4c35-9949-adda70ae20c7"
-					(reference "TP17")
+					(reference "TP_LO")
 					(unit 1)
 				)
@@
 		(on_board yes)
 		(dnp no)
-		(property "Reference" "TP18"
+		(property "Reference" "TP_HI"
 			(at 233.68 40.64 90)
 			(effects
@@
 			(project "BitshokaNiniV1.1"
 				(path "/e63e39d7-6ac0-4ffd-8aa3-1841a4541b55/4cf9c075-d009-4c35-9949-adda70ae20c7"
-					(reference "TP18")
+					(reference "TP_HI")
 					(unit 1)
 				)
@@
 		(on_board yes)
 		(dnp no)
-		(property "Reference" "TP16"
-			(at 187.96 35.56 90)
+		(property "Reference" "TXD_LO"
+			(at 186.69 35.56 90)
 			(effects
 				(font
@@
 			(project "BitshokaNiniV1.1"
 				(path "/e63e39d7-6ac0-4ffd-8aa3-1841a4541b55/4cf9c075-d009-4c35-9949-adda70ae20c7"
-					(reference "TP16")
+					(reference "TXD_LO")
 					(unit 1)
 				)
@@
 		(on_board yes)
 		(dnp no)
-		(property "Reference" "TP12"
+		(property "Reference" "TXD"
 			(at 62.23 104.14 90)
 			(effects
@@
 			(project "BitshokaNiniV1.1"
 				(path "/e63e39d7-6ac0-4ffd-8aa3-1841a4541b55/4cf9c075-d009-4c35-9949-adda70ae20c7"
-					(reference "TP12")
+					(reference "TXD")
 					(unit 1)
 				)

Commit message: Manfacturing prep
Add part numbers and did initial BOM optimization (Hope to do more after testing)
Created Manufacturing files
Parts:
- added C35: 100uF, Capacitor_SMD:C_1206_3216Metric, symbol Device:C
- C28: value C_Small -> 0.1uF
- C31: value 0.1uF? -> 0.1uF
- C43: DK 1276-1782-1-ND -> (none); PARTNO CL31A107MQHNNNE -> (none)
- R21: value 20k -> 10k
- R28: value 440 -> 442
- R29: value 550 -> 549
- R30: value 500 -> 499
- R31: value 335 -> 332
- R32: value 400 -> 402
- renumbered 0.9V to 0.9V1, TP22 to CLK1, CTSI to CTSI1, DIR_HI to DIR_HI1, DIR_LO to DIR_LO1, TP_HI to HI1, TP_LO to LO1, RST to RST1, RST_LO to RST_LO1, RXD to RXD1, RXD to RXD2, TXD to TXD1, TXD to TXD2, TXD_LO to TXD_LO1
Connections:
- net GND: now also C35.2; no longer LO1.1
- net VDD: now also C35.1
- net at R17.2, U9.6 (A4): now also LO1.1
Other:
- note added: "Need to confirm C28 & C31 value"
- note added: "Need to confirm R33 & R34 and the voltage divider"
- moved on the sheet: 0.9V1, C33, CTSI1, DIR_HI1, DIR_LO1, LO1, Q1, R17, R36, R37, RST_DET1, RXD2

Commit message: New Inductor & BOM fix
Changed the inductor and cleaned up files for JLCPCB order.
Other:
- moved on the sheet: 1V8, C30
Changed lines of the file:
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@@
 	)
 	(junction
-		(at 57.15 29.21)
+		(at 66.04 29.21)
 		(diameter 0.9144)
 		(color 0 0 0 0)
@@
 	(wire
 		(pts
+			(xy 46.99 43.18) (xy 66.04 43.18)
+		)
+		(stroke
+			(width 0)
+			(type solid)
+		)
+	)
+	(wire
+		(pts
 			(xy 242.57 29.21) (xy 242.57 35.56)
 		)
@@
 	(wire
 		(pts
-			(xy 57.15 39.37) (xy 57.15 43.18)
+			(xy 66.04 39.37) (xy 66.04 43.18)
 		)
 		(stroke
@@
 	(wire
 		(pts
-			(xy 46.99 43.18) (xy 57.15 43.18)
-		)
-		(stroke
-			(width 0)
-			(type solid)
-		)
-	)
-	(wire
-		(pts
 			(xy 119.38 114.3) (xy 142.24 114.3)
 		)
@@
 	(wire
 		(pts
+			(xy 54.61 29.21) (xy 66.04 29.21)
+		)
+		(stroke
+			(width 0)
+			(type solid)
+		)
+	)
+	(wire
+		(pts
 			(xy 35.56 39.37) (xy 35.56 43.18)
 		)
@@
 	(wire
 		(pts
-			(xy 54.61 29.21) (xy 57.15 29.21)
-		)
-		(stroke
-			(width 0)
-			(type solid)
-		)
-	)
-	(wire
-		(pts
 			(xy 181.61 29.21) (xy 204.47 29.21)
 		)
@@
 	(wire
 		(pts
-			(xy 57.15 29.21) (xy 60.96 29.21)
+			(xy 66.04 29.21) (xy 69.85 29.21)
 		)
 		(stroke
@@
 	(wire
 		(pts
-			(xy 57.15 29.21) (xy 57.15 31.75)
+			(xy 66.04 29.21) (xy 66.04 31.75)
 		)
 		(stroke
@@
 	)
 	(label "1V8"
-		(at 57.15 29.21 0)
+		(at 66.04 29.21 0)
 		(effects
 			(font
@@
 	(symbol
 		(lib_id "Device:C")
-		(at 57.15 35.56 0)
+		(at 66.04 35.56 0)
 		(unit 1)
 		(exclude_from_sim no)
@@
 		(dnp no)
 		(property "Reference" "C30"
-			(at 58.42 33.655 0)
+			(at 67.31 33.655 0)
 			(effects
 				(font
@@
 		)
 		(property "Value" "1uF"
-			(at 59.055 39.37 0)
+			(at 67.945 39.37 0)
 			(effects
 				(font
@@
 		)
 		(property "Footprint" "Capacitor_SMD:C_0402_1005Metric"
-			(at 57.15 35.56 0)
+			(at 66.04 35.56 0)
 			(effects
 				(font
@@
 		)
 		(property "Datasheet" "~"
-			(at 57.15 35.56 0)
+			(at 66.04 35.56 0)
 			(effects
 				(font
@@
 		)
 		(property "Description" "Unpolarized capacitor"
-			(at 57.15 35.56 0)
+			(at 66.04 35.56 0)
 			(effects
 				(font
@@
 		)
 		(property "DK" "587-5514-1-ND"
-			(at 57.15 35.56 0)
+			(at 66.04 35.56 0)
 			(effects
 				(font
@@
 		)
 		(property "PARTNO" "EMK105BJ105MV-F"
-			(at 57.15 35.56 0)
+			(at 66.04 35.56 0)
 			(effects
 				(font
@@
 	(symbol
 		(lib_id "Connector:TestPoint")
-		(at 60.96 29.21 270)
+		(at 69.85 29.21 270)
 		(mirror x)
 		(unit 1)
@@
 		(dnp no)
 		(property "Reference" "1V8"
-			(at 67.31 29.21 90)
+			(at 76.2 29.21 90)
 			(effects
 				(font
@@
 		)
 		(property "Value" "TestPoint"
-			(at 66.675 27.9401 90)
+			(at 75.565 27.9401 90)
 			(effects
 				(font
@@
 		)
 		(property "Footprint" "TestPoint:TestPoint_Pad_D1.5mm"
-			(at 60.96 24.13 0)
+			(at 69.85 24.13 0)
 			(effects
 				(font
@@
 		)
 		(property "Datasheet" "~"
-			(at 60.96 24.13 0)
+			(at 69.85 24.13 0)
 			(effects
 				(font
@@
 		)
 		(property "Description" "test point"
-			(at 60.96 29.21 0)
+			(at 69.85 29.21 0)
 			(effects
 				(font

Commit message: Fixed CMOS clock
Parts:
- U7: LCSC C5137262 -> (none); PARTNO SX3M25.000E20F30THN -> SX3M24.000E20F30THN
Changed lines of the file:
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@@
 			)
 		)
-		(property "PARTNO" "SX3M25.000E20F30THN"
+		(property "PARTNO" "SX3M24.000E20F30THN"
 			(at 41.91 171.45 0)
 			(effects
@@
 			)
 		)
-		(property "LCSC" "C5137262"
+		(property "LCSC" ""
 			(at 41.91 171.45 0)
 			(effects
